File: analog front-end/4Input-1Output_board/Schematics_PCB/schematic3.sch (KiCad schematic (older format))
At the start: 37 parts, among them J1 Screw_Terminal_1x04, J2 Screw_Terminal_1x08, J3 Screw_Terminal_1x08, J4 Screw_Terminal_1x03, J5 Screw_Terminal_1x12, J6 Screw_Terminal_1x08, J7 Screw_Terminal_1x08, U1 INA128, U2 INA128, U3 INA128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

Commit message: Started KiCAD schematics of all the analog part of the Teensy-EIS.
Parts:
- RV1, RV2, RV3, RV4: symbol POT -> POT-RESCUE-schematic3
Changed lines of the file:
@@
 EESchema Schematic File Version 2
+LIBS:schematic3-rescue
 LIBS:power
 LIBS:device
@@
 4 INAs board\ntwo bypass caps in the beginning of the power rails and two caps for every opas\nEvery INA has screw terminals so we can easy jump everywhere with cables\nEvery INA has no or adjustable gain\nEvery INA has a double set of screw inputs\n\nBetween the first screw and the second screw\na resistor can be placed.\nThese resistors can be used for filtering \nor using 2/3 terminals for summing signals\n
 $Comp
-L POT RV1
+L POT-RESCUE-schematic3 RV1
 U 1 1 587905FA
 P 3350 3550
@@
 	3950 3700 3950 3800
 $Comp
-L POT RV2
+L POT-RESCUE-schematic3 RV2
 U 1 1 587FBB8E
 P 3950 3550
@@
 	4500 3700 4500 3800
 $Comp
-L POT RV3
+L POT-RESCUE-schematic3 RV3
 U 1 1 587FBC8F
 P 4500 3550
@@
 	5100 3700 5100 3800
 $Comp
-L POT RV4
+L POT-RESCUE-schematic3 RV4
 U 1 1 588077DE
 P 5100 3550
