File: analog front-end/Design_schematics/Complete_analog_front-end.sch (KiCad schematic (older format))
At the start: 10 parts

Commit message: Functional diagram of the project is finished. Few details are missing: pull-down resistor, position of the filter capacitor...
Parts:
- removed P? (x2): BNC, symbol BNC
- removed Q?: Q_NPN_BCE, symbol Q_NPN_BCE
- removed RV?: POT, symbol POT
- removed SW?: SWITCH_INV, symbol SWITCH_INV
- removed U? (x3): INA128, symbol INA128
- removed U?: NMA0515SC, Converters_DCDC_ACDC:DCDC-Conv_muRata_NMAxxxxSC, symbol NMA0515SC
- gave numbers to parts that had none: 1
Connections:
- net DAC_reference is gone; now on net ADC input/DAC_reference: U5.38 (A22_DAC1)
- net DAC_signal is gone; now on net analog_DAC/DAC_signal: U5.37 (A21_DAC0)
- net ADC input/ADC_input1: now also U5.50 (23_A9_PWM_Touch)
- net analog_DAC/EnableOutput: now reaches U5.16 (24)
- net ADC input/ADC_input2: now reaches U5.35 (38_A19_PWM_SDA1)
- no-connect marks 2 -> 81
Other:
- note added: "Functional diagram of the connections between the Teensy, the power stage,\n and the analog frontend"
- note added: "The details of the INAs board are in "4Input-1Output_board"."
