File: analog front-end/Design_schematics/analog_DAC.sch (KiCad schematic (older format))
At the start: 12 parts, among them K1 RELAY_2RT, P6 BNC, Q1 Q_NPN_BCE, U10 INA128, U8 INA128, U9 INA128

Commit message: Fix shutdown. Now there is a 47 kOhm pulldown resitor and the relayPin goes low.
Parts:
- PullDown1: value R -> 47 k
Changed lines of the file:
@@
 P 7950 4250
 F 0 "PullDown1" V 8030 4250 50  0000 C CNN
-F 1 "R" V 7950 4250 50  0000 C CNN
+F 1 "47 k" V 7950 4250 50  0000 C CNN
 F 2 "" V 7880 4250 50  0000 C CNN
 F 3 "" H 7950 4250 50  0000 C CNN
